Commit message: Add files via upload

File: agribot_testing_3_description/urdf/agribot_testing_3.xacro (robot description, xacro)
@@ -6,5 +6,5 @@
 <link name="base_link">
   <inertial>
-    <origin xyz="-0.2350880604034246 0.06665534217761451 0.2751777756723828" rpy="0 0 0"/>
+    <origin xyz="-0.2350880604034247 0.06665534217761437 0.38865777567238247" rpy="0 0 0"/>
     <mass value="33.861613005474375"/>
     <inertia ixx="1.628198" iyy="2.74751" izz="3.065301" ixy="-0.000154" iyz="-0.001994" ixz="-0.003471"/>
@@ -26,10 +26,10 @@
 <link name="wheel_attachment_v3_1">
   <inertial>
-    <origin xyz="3.8128879042975683e-07 -0.019174361968348597 -3.432632603838498e-07" rpy="0 0 0"/>
+    <origin xyz="3.8128879042975683e-07 -0.019174361968348846 -3.4326326046885125e-07" rpy="0 0 0"/>
     <mass value="2.8820189071853717"/>
-    <inertia ixx="0.010501" iyy="0.020705" izz="0.010501" ixy="0.0" iyz="-0.0" ixz="-0.0"/>
-  </inertial>
-  <visual>
-    <origin xyz="0.607089 0.154579 0.014853" rpy="0 0 0"/>
+    <inertia ixx="0.010501" iyy="0.020705" izz="0.010501" ixy="0.0" iyz="-0.0" ixz="0.0"/>
+  </inertial>
+  <visual>
+    <origin xyz="0.607089 0.154579 -0.098627" rpy="0 0 0"/>
     <geometry>
       <mesh filename="package://agribot_testing_3_description/meshes/wheel_attachment_v3_1.stl" scale="0.001 0.001 0.001"/>
@@ -38,5 +38,5 @@
   </visual>
   <collision>
-    <origin xyz="0.607089 0.154579 0.014853" rpy="0 0 0"/>
+    <origin xyz="0.607089 0.154579 -0.098627" rpy="0 0 0"/>
     <geometry>
       <mesh filename="package://agribot_testing_3_description/meshes/wheel_attachment_v3_1.stl" scale="0.001 0.001 0.001"/>
@@ -46,10 +46,10 @@
 <link name="wheel_attachment_v5_1">
   <inertial>
-    <origin xyz="-3.348505955846903e-07 -0.019183612949765283 3.802777481676928e-07" rpy="0 0 0"/>
+    <origin xyz="-3.348505955291792e-07 -0.019183612949765505 3.8027774791615787e-07" rpy="0 0 0"/>
     <mass value="2.8568879657816306"/>
     <inertia ixx="0.0105" iyy="0.020703" izz="0.0105" ixy="0.0" iyz="-0.0" ixz="-0.0"/>
   </inertial>
   <visual>
-    <origin xyz="-0.137665 0.154179 0.01188" rpy="0 0 0"/>
+    <origin xyz="-0.137665 0.154179 -0.1016" rpy="0 0 0"/>
     <geometry>
       <mesh filename="package://agribot_testing_3_description/meshes/wheel_attachment_v5_1.stl" scale="0.001 0.001 0.001"/>
@@ -58,5 +58,5 @@
   </visual>
   <collision>
-    <origin xyz="-0.137665 0.154179 0.01188" rpy="0 0 0"/>
+    <origin xyz="-0.137665 0.154179 -0.1016" rpy="0 0 0"/>
     <geometry>
       <mesh filename="package://agribot_testing_3_description/meshes/wheel_attachment_v5_1.stl" scale="0.001 0.001 0.001"/>
@@ -66,10 +66,10 @@
 <link name="wheel_attachment_v5_2">
   <inertial>
-    <origin xyz="-4.557887117728754e-07 0.01918397188057064 1.3545067892827e-07" rpy="0 0 0"/>
+    <origin xyz="-4.557887117728754e-07 0.019183971880570305 1.354506786177545e-07" rpy="0 0 0"/>
     <mass value="2.8568879657816306"/>
     <inertia ixx="0.0105" iyy="0.020703" izz="0.0105" ixy="0.0" iyz="-0.0" ixz="0.0"/>
   </inertial>
   <visual>
-    <origin xyz="0.607599 -0.287008 0.013466" rpy="0 0 0"/>
+    <origin xyz="0.607599 -0.287008 -0.100014" rpy="0 0 0"/>
     <geometry>
       <mesh filename="package://agribot_testing_3_description/meshes/wheel_attachment_v5_2.stl" scale="0.001 0.001 0.001"/>
@@ -78,5 +78,5 @@
   </visual>
   <collision>
-    <origin xyz="0.607599 -0.287008 0.013466" rpy="0 0 0"/>
+    <origin xyz="0.607599 -0.287008 -0.100014" rpy="0 0 0"/>
     <geometry>
       <mesh filename="package://agribot_testing_3_description/meshes/wheel_attachment_v5_2.stl" scale="0.001 0.001 0.001"/>
@@ -86,10 +86,10 @@
 <link name="wheel_attachment_v5_3">
   <inertial>
-    <origin xyz="3.728495584776059e-07 0.019183971880533668 -3.65455947405266e-07" rpy="0 0 0"/>
+    <origin xyz="3.728495583943392e-07 0.019183971880533446 -3.6545594768455647e-07" rpy="0 0 0"/>
     <mass value="2.8568879657816306"/>
     <inertia ixx="0.0105" iyy="0.020703" izz="0.0105" ixy="0.0" iyz="-0.0" ixz="0.0"/>
   </inertial>
   <visual>
-    <origin xyz="-0.137524 -0.287008 0.011905" rpy="0 0 0"/>
+    <origin xyz="-0.137524 -0.287008 -0.101575" rpy="0 0 0"/>
     <geometry>
       <mesh filename="package://agribot_testing_3_description/meshes/wheel_attachment_v5_3.stl" scale="0.001 0.001 0.001"/>
@@ -98,5 +98,5 @@
   </visual>
   <collision>
-    <origin xyz="-0.137524 -0.287008 0.011905" rpy="0 0 0"/>
+    <origin xyz="-0.137524 -0.287008 -0.101575" rpy="0 0 0"/>
     <geometry>
       <mesh filename="package://agribot_testing_3_description/meshes/wheel_attachment_v5_3.stl" scale="0.001 0.001 0.001"/>
@@ -106,10 +106,10 @@
 <link name="ydlidar_x4_v1_1">
   <inertial>
-    <origin xyz="-0.0017058707003289666 -3.205345905643586e-07 0.020201312343200273" rpy="0 0 0"/>
+    <origin xyz="-0.0017058707003289857 -3.2053459074476987e-07 0.020201312343200217" rpy="0 0 0"/>
     <mass value="1.1515616542314233"/>
     <inertia ixx="0.000489" iyy="0.000861" izz="0.000987" ixy="0.0" iyz="0.0" ixz="0.000148"/>
   </inertial>
   <visual>
-    <origin xyz="-0.014827 -0.066215 -0.439932" rpy="0 0 0"/>
+    <origin xyz="-0.014827 -0.066215 -0.553412" rpy="0 0 0"/>
     <geometry>
       <mesh filename="package://agribot_testing_3_description/meshes/ydlidar_x4_v1_1.stl" scale="0.001 0.001 0.001"/>
@@ -118,5 +118,5 @@
   </visual>
   <collision>
-    <origin xyz="-0.014827 -0.066215 -0.439932" rpy="0 0 0"/>
+    <origin xyz="-0.014827 -0.066215 -0.553412" rpy="0 0 0"/>
     <geometry>
       <mesh filename="package://agribot_testing_3_description/meshes/ydlidar_x4_v1_1.stl" scale="0.001 0.001 0.001"/>
@@ -126,10 +126,10 @@
 <link name="camera_mount_v1_1">
   <inertial>
-    <origin xyz="0.01250002972934782 -0.012500320534587647 0.07788741036522173" rpy="0 0 0"/>
+    <origin xyz="0.012500029729347837 -0.012500320534587814 0.07788741036522173" rpy="0 0 0"/>
     <mass value="0.5409900233067988"/>
     <inertia ixx="0.000886" iyy="0.00104" izz="0.00081" ixy="-0.000133" iyz="-0.0" ixz="0.0"/>
   </inertial>
   <visual>
-    <origin xyz="0.010173 0.088785 -0.439932" rpy="0 0 0"/>
+    <origin xyz="0.010173 0.088785 -0.553412" rpy="0 0 0"/>
     <geometry>
       <mesh filename="package://agribot_testing_3_description/meshes/camera_mount_v1_1.stl" scale="0.001 0.001 0.001"/>
@@ -138,5 +138,5 @@
   </visual>
   <collision>
-    <origin xyz="0.010173 0.088785 -0.439932" rpy="0 0 0"/>
+    <origin xyz="0.010173 0.088785 -0.553412" rpy="0 0 0"/>
     <geometry>
       <mesh filename="package://agribot_testing_3_description/meshes/camera_mount_v1_1.stl" scale="0.001 0.001 0.001"/>
@@ -146,10 +146,10 @@
 <link name="kinectv2_v1_1">
   <inertial>
-    <origin xyz="0.00021058727276473174 -0.00269160106068711 0.038314477205350084" rpy="0 0 0"/>
+    <origin xyz="0.00021058727276470398 -0.0026916010606874013 0.03831447720534975" rpy="0 0 0"/>
     <mass value="0.7810524514781609"/>
     <inertia ixx="0.001383" iyy="0.002954" izz="0.003916" ixy="-0.001402" iyz="2.1e-05" ixz="-1.1e-05"/>
   </inertial>
   <visual>
-    <origin xyz="-0.002327 0.101285 -0.542432" rpy="0 0 0"/>
+    <origin xyz="-0.002327 0.101285 -0.655912" rpy="0 0 0"/>
     <geometry>
       <mesh filename="package://agribot_testing_3_description/meshes/kinectv2_v1_1.stl" scale="0.001 0.001 0.001"/>
@@ -158,5 +158,5 @@
   </visual>
   <collision>
-    <origin xyz="-0.002327 0.101285 -0.542432" rpy="0 0 0"/>
+    <origin xyz="-0.002327 0.101285 -0.655912" rpy="0 0 0"/>
     <geometry>
       <mesh filename="package://agribot_testing_3_description/meshes/kinectv2_v1_1.stl" scale="0.001 0.001 0.001"/>
@@ -166,10 +166,10 @@
 <link name="base_arm_v2_1">
   <inertial>
-    <origin xyz="2.9729364636743583e-08 0.01249967946542374 0.010307514282643648" rpy="0 0 0"/>
+    <origin xyz="2.972936491429934e-08 0.01249967946542388 0.010307514282643426" rpy="0 0 0"/>
     <mass value="0.9330886709339293"/>
-    <inertia ixx="0.001421" iyy="0.001421" izz="0.002578" ixy="0.0" iyz="0.0" ixz="-0.0"/>
-  </inertial>
-  <visual>
-    <origin xyz="0.460173 -0.221215 -0.439932" rpy="0 0 0"/>
+    <inertia ixx="0.001421" iyy="0.001421" izz="0.002578" ixy="-0.0" iyz="0.0" ixz="0.0"/>
+  </inertial>
+  <visual>
+    <origin xyz="0.460173 -0.221215 -0.553412" rpy="0 0 0"/>
     <geometry>
       <mesh filename="package://agribot_testing_3_description/meshes/base_arm_v2_1.stl" scale="0.001 0.001 0.001"/>
@@ -178,5 +178,5 @@
   </visual>
   <collision>
-    <origin xyz="0.460173 -0.221215 -0.439932" rpy="0 0 0"/>
+    <origin xyz="0.460173 -0.221215 -0.553412" rpy="0 0 0"/>
     <geometry>
       <mesh filename="package://agribot_testing_3_description/meshes/base_arm_v2_1.stl" scale="0.001 0.001 0.001"/>
@@ -186,17 +186,17 @@
 <link name="link_1_v3_1">
   <inertial>
-    <origin xyz="-0.003271917210980746 0.004456357998370242 0.025593960333273658" rpy="0 0 0"/>
+    <origin xyz="-0.003271917210980857 0.004456357998369992 0.025593960333273547" rpy="0 0 0"/>
     <mass value="1.6613467153005188"/>
     <inertia ixx="0.002663" iyy="0.002483" izz="0.002146" ixy="-2.2e-05" iyz="-0.000454" ixz="0.000339"/>
   </inertial>
   <visual>
-    <origin xyz="0.460173 -0.233715 -0.480932" rpy="0 0 0"/>
+    <origin xyz="0.460173 -0.233715 -0.594412" rpy="0 0 0"/>
     <geometry>
       <mesh filename="package://agribot_testing_3_description/meshes/link_1_v3_1.stl" scale="0.001 0.001 0.001"/>
     </geometry>
-    <material name="opaque646464"/>
-  </visual>
-  <collision>
-    <origin xyz="0.460173 -0.233715 -0.480932" rpy="0 0 0"/>
+    <material name="opaque636363"/>
+  </visual>
+  <collision>
+    <origin xyz="0.460173 -0.233715 -0.594412" rpy="0 0 0"/>
     <geometry>
       <mesh filename="package://agribot_testing_3_description/meshes/link_1_v3_1.stl" scale="0.001 0.001 0.001"/>
@@ -206,10 +206,10 @@
 <link name="link_2_v1_1">
   <inertial>
-    <origin xyz="0.0004995698471454424 0.05852714517882579 0.055084304746622625" rpy="0 0 0"/>
+    <origin xyz="0.0004995698471453314 0.05852714517882551 0.055084304746622736" rpy="0 0 0"/>
     <mass value="0.2532575834482899"/>
-    <inertia ixx="0.000795" iyy="0.000454" izz="0.000342" ixy="0.0" iyz="-0.000362" ixz="0.0"/>
-  </inertial>
-  <visual>
-    <origin xyz="0.468884 -0.274766 -0.555672" rpy="0 0 0"/>
+    <inertia ixx="0.000795" iyy="0.000454" izz="0.000342" ixy="-0.0" iyz="-0.000362" ixz="0.0"/>
+  </inertial>
+  <visual>
+    <origin xyz="0.468884 -0.274766 -0.669152" rpy="0 0 0"/>
     <geometry>
       <mesh filename="package://agribot_testing_3_description/meshes/link_2_v1_1.stl" scale="0.001 0.001 0.001"/>
@@ -218,5 +218,5 @@
   </visual>
   <collision>
-    <origin xyz="0.468884 -0.274766 -0.555672" rpy="0 0 0"/>
+    <origin xyz="0.468884 -0.274766 -0.669152" rpy="0 0 0"/>
     <geometry>
       <mesh filename="package://agribot_testing_3_description/meshes/link_2_v1_1.stl" scale="0.001 0.001 0.001"/>
@@ -226,10 +226,10 @@
 <link name="link_3_v2_1">
   <inertial>
-    <origin xyz="0.018953081069860656 0.03419477091099504 0.03607507426293899" rpy="0 0 0"/>
+    <origin xyz="0.018953081069860656 0.03419477091099454 0.0360750742629391" rpy="0 0 0"/>
     <mass value="0.6682248227150334"/>
     <inertia ixx="0.002549" iyy="0.001313" izz="0.001356" ixy="-6e-06" iyz="-0.001236" ixz="-7e-06"/>
   </inertial>
   <visual>
-    <origin xyz="0.465884 -0.394167 -0.675073" rpy="0 0 0"/>
+    <origin xyz="0.465884 -0.394167 -0.788553" rpy="0 0 0"/>
     <geometry>
       <mesh filename="package://agribot_testing_3_description/meshes/link_3_v2_1.stl" scale="0.001 0.001 0.001"/>
@@ -238,5 +238,5 @@
   </visual>
   <collision>
-    <origin xyz="0.465884 -0.394167 -0.675073" rpy="0 0 0"/>
+    <origin xyz="0.465884 -0.394167 -0.788553" rpy="0 0 0"/>
     <geometry>
       <mesh filename="package://agribot_testing_3_description/meshes/link_3_v2_1.stl" scale="0.001 0.001 0.001"/>
@@ -246,10 +246,10 @@
 <link name="eef_base_v1_1">
   <inertial>
-    <origin xyz="-0.018914256538726415 0.043186333490104034 0.004331187030702122" rpy="0 0 0"/>
+    <origin xyz="-0.018914256538726526 0.04318633349010392 0.004331187030702122" rpy="0 0 0"/>
     <mass value="0.33153308863416847"/>
     <inertia ixx="9.1e-05" iyy="9.2e-05" izz="0.000121" ixy="-0.0" iyz="-5e-06" ixz="-1e-06"/>
   </inertial>
   <visual>
-    <origin xyz="0.427784 -0.484622 -0.765528" rpy="0 0 0"/>
+    <origin xyz="0.427784 -0.484622 -0.879008" rpy="0 0 0"/>
     <geometry>
       <mesh filename="package://agribot_testing_3_description/meshes/eef_base_v1_1.stl" scale="0.001 0.001 0.001"/>
@@ -258,5 +258,5 @@
   </visual>
   <collision>
-    <origin xyz="0.427784 -0.484622 -0.765528" rpy="0 0 0"/>
+    <origin xyz="0.427784 -0.484622 -0.879008" rpy="0 0 0"/>
     <geometry>
       <mesh filename="package://agribot_testing_3_description/meshes/eef_base_v1_1.stl" scale="0.001 0.001 0.001"/>
@@ -266,10 +266,10 @@
 <link name="left_claw_v3_1">
   <inertial>
-    <origin xyz="-0.03162572015420595 0.056519004177445376 0.0008015719343229533" rpy="0 0 0"/>
+    <origin xyz="-0.03162572015420595 0.056519004177445153 0.0008015719343230643" rpy="0 0 0"/>
     <mass value="0.02736131598910003"/>
     <inertia ixx="2.2e-05" iyy="5e-06" izz="2.7e-05" ixy="9e-06" iyz="-0.0" ixz="0.0"/>
   </inertial>
   <visual>
-    <origin xyz="0.478294 -0.529558 -0.756071" rpy="0 0 0"/>
+    <origin xyz="0.478294 -0.529558 -0.869551" rpy="0 0 0"/>
     <geometry>
       <mesh filename="package://agribot_testing_3_description/meshes/left_claw_v3_1.stl" scale="0.001 0.001 0.001"/>
@@ -278,5 +278,5 @@
   </visual>
   <collision>
-    <origin xyz="0.478294 -0.529558 -0.756071" rpy="0 0 0"/>
+    <origin xyz="0.478294 -0.529558 -0.869551" rpy="0 0 0"/>
     <geometry>
       <mesh filename="package://agribot_testing_3_description/meshes/left_claw_v3_1.stl" scale="0.001 0.001 0.001"/>
@@ -286,10 +286,10 @@
 <link name="right_claw_v3_1">
   <inertial>
-    <origin xyz="0.03162000829220274 0.056523865138236706 0.0008015719343187344" rpy="0 0 0"/>
+    <origin xyz="0.03162000829220274 0.05652386513823637 0.0008015719343187344" rpy="0 0 0"/>
     <mass value="0.027361315989100486"/>
     <inertia ixx="2.2e-05" iyy="5e-06" izz="2.7e-05" ixy="-9e-06" iyz="-0.0" ixz="-0.0"/>
   </inertial>
   <visual>
-    <origin xyz="0.415294 -0.529558 -0.756071" rpy="0 0 0"/>
+    <origin xyz="0.415294 -0.529558 -0.869551" rpy="0 0 0"/>
     <geometry>
       <mesh filename="package://agribot_testing_3_description/meshes/right_claw_v3_1.stl" scale="0.001 0.001 0.001"/>
@@ -298,5 +298,5 @@
   </visual>
   <collision>
-    <origin xyz="0.415294 -0.529558 -0.756071" rpy="0 0 0"/>
+    <origin xyz="0.415294 -0.529558 -0.869551" rpy="0 0 0"/>
     <geometry>
       <mesh filename="package://agribot_testing_3_description/meshes/right_claw_v3_1.stl" scale="0.001 0.001 0.001"/>
@@ -305,5 +305,5 @@
 </link>
 <joint name="back_right" type="continuous">
-  <origin xyz="-0.607089 -0.154579 -0.014853" rpy="0 0 0"/>
+  <origin xyz="-0.607089 -0.154579 0.098627" rpy="0 0 0"/>
   <parent link="base_link"/>
   <child link="wheel_attachment_v3_1"/>
@@ -311,5 +311,5 @@
 </joint>
 <joint name="front_right" type="continuous">
-  <origin xyz="0.137665 -0.154179 -0.01188" rpy="0 0 0"/>
+  <origin xyz="0.137665 -0.154179 0.1016" rpy="0 0 0"/>
   <parent link="base_link"/>
   <child link="wheel_attachment_v5_1"/>
@@ -317,5 +317,5 @@
 </joint>
 <joint name="back_left" type="continuous">
-  <origin xyz="-0.607599 0.287008 -0.013466" rpy="0 0 0"/>
+  <origin xyz="-0.607599 0.287008 0.100014" rpy="0 0 0"/>
   <parent link="base_link"/>
   <child link="wheel_attachment_v5_2"/>
@@ -323,5 +323,5 @@
 </joint>
 <joint name="front_left" type="continuous">
-  <origin xyz="0.137524 0.287008 -0.011905" rpy="0 0 0"/>
+  <origin xyz="0.137524 0.287008 0.101575" rpy="0 0 0"/>
   <parent link="base_link"/>
   <child link="wheel_attachment_v5_3"/>
@@ -329,10 +329,10 @@
 </joint>
 <joint name="Rigid 8" type="fixed">
-  <origin xyz="0.014827 0.066215 0.439932" rpy="0 0 0"/>
+  <origin xyz="0.014827 0.066215 0.553412" rpy="0 0 0"/>
   <parent link="base_link"/>
   <child link="ydlidar_x4_v1_1"/>
 </joint>
 <joint name="Rigid 9" type="fixed">
-  <origin xyz="-0.010173 -0.088785 0.439932" rpy="0 0 0"/>
+  <origin xyz="-0.010173 -0.088785 0.553412" rpy="0 0 0"/>
   <parent link="base_link"/>
   <child link="camera_mount_v1_1"/>
@@ -344,5 +344,5 @@
 </joint>
 <joint name="Rigid 11" type="fixed">
-  <origin xyz="-0.460173 0.221215 0.439932" rpy="0 0 0"/>
+  <origin xyz="-0.460173 0.221215 0.553412" rpy="0 0 0"/>
   <parent link="base_link"/>
   <child link="base_arm_v2_1"/>

File: agribot_testing_3_description/urdf/materials.xacro (robot description, xacro)
@@ -7,5 +7,5 @@
   <color rgba="0.6274509803921569 0.6274509803921569 0.6274509803921569 1.0"/>
 </material>
-<material name="opaque646464">
+<material name="opaque636363">
   <color rgba="0.25098039215686274 0.25098039215686274 0.25098039215686274 1.0"/>
 </material>

Commit message: configured files for gazebo

File: agribot_testing_3_description/urdf/agribot_testing_3.xacro (robot description, xacro)
@@ -164,4 +164,11 @@
   </collision>
 </link>
+<link name="optical_frame"/>
+<joint name="kinect_optical_frame" type="fixed">
+  <parent link="kinectv2_v1_1"/>
+  <child link="optical_frame"/>
+  <origin xyz="0 0 0" rpy="-1.5708 0 -1.5708"/>
+  <axis xyz="0 0 0"/>
+</joint>
 <link name="base_arm_v2_1">
   <inertial>

Commit message: corrected frames

File: agribot_testing_3_description/urdf/agribot_testing_3.xacro (robot description, xacro)
@@ -111,5 +111,5 @@
   </inertial>
   <visual>
-    <origin xyz="-0.014827 -0.066215 -0.553412" rpy="0 0 0"/>
+    <origin xyz="-0.014827 -0.066215 -0.583412" rpy="0 0 0"/>
     <geometry>
       <mesh filename="package://agribot_testing_3_description/meshes/ydlidar_x4_v1_1.stl" scale="0.001 0.001 0.001"/>
@@ -168,5 +168,5 @@
   <parent link="kinectv2_v1_1"/>
   <child link="optical_frame"/>
-  <origin xyz="0 0 0" rpy="-1.5708 0 -1.5708"/>
+  <origin xyz="0.1 0 0.0375" rpy="-1.5708 0 0.5236"/>false
   <axis xyz="0 0 0"/>
 </joint>
@@ -315,5 +315,5 @@
   <parent link="base_link"/>
   <child link="wheel_attachment_v3_1"/>
-  <axis xyz="-0.0 -1.0 0.0"/>
+  <axis xyz="-0.0 1.0 0.0"/>
 </joint>
 <joint name="front_right" type="continuous">
@@ -321,5 +321,5 @@
   <parent link="base_link"/>
   <child link="wheel_attachment_v5_1"/>
-  <axis xyz="-0.0 -1.0 0.0"/>
+  <axis xyz="-0.0 1.0 0.0"/>
 </joint>
 <joint name="back_left" type="continuous">
@@ -336,5 +336,5 @@
 </joint>
 <joint name="Rigid 8" type="fixed">
-  <origin xyz="0.014827 0.066215 0.553412" rpy="0 0 0"/>
+  <origin xyz="0.014827 0.066215 0.583412" rpy="0 0 0"/>
   <parent link="base_link"/>
   <child link="ydlidar_x4_v1_1"/>

Commit message: corrected frames

File: agribot_testing_3_description/urdf/agribot_testing_3.xacro (robot description, xacro)
@@ -164,9 +164,16 @@
   </collision>
 </link>
+<link name="rgb_frame"/>
+<joint name="kinect_rgb_frame" type="fixed">
+  <parent link="kinectv2_v1_1"/>
+  <child link="rgb_frame"/>
+  <origin xyz="0.075 0.075 0.0375" rpy="0 0 2.0944"/>
+  <axis xyz="0 0 0"/>
+</joint>
 <link name="optical_frame"/>
-<joint name="kinect_optical_frame" type="fixed">
-  <parent link="kinectv2_v1_1"/>
+<joint name="rgb_optical_frame" type="fixed">
+  <parent link="rgb_frame"/>
   <child link="optical_frame"/>
-  <origin xyz="0.1 0 0.0375" rpy="-1.5708 0 0.5236"/>false
+  <origin xyz="0 0 0" rpy="-1.5708 0 -1.5708"/>
   <axis xyz="0 0 0"/>
 </joint>
