Commit message: Add files via upload

File: agribot_v4_description/urdf/agribot_v4.xacro (robot description, xacro)
@@ -255,5 +255,5 @@
       <mesh filename="package://agribot_v4_description/meshes/link_1_v3_1.stl" scale="0.001 0.001 0.001"/>
     </geometry>
-    <material name="opaque636363"/>
+    <material name="opaque272727"/>
   </visual>
   <collision>
@@ -384,5 +384,5 @@
   </collision>
 </link>
-<joint name="Revolute 1" type="continuous">
+<joint name="front_right_steer" type="continuous">
   <origin xyz="0.372581 -0.24075 0.2316" rpy="0 0 0"/>
   <parent link="base_link"/>
@@ -390,5 +390,5 @@
   <axis xyz="0.002015 0.0 -0.999998"/>
 </joint>
-<joint name="Revolute 2" type="continuous">
+<joint name="front_left_steer" type="continuous">
   <origin xyz="0.372522 0.24115 0.231574" rpy="0 0 0"/>
   <parent link="base_link"/>
@@ -396,5 +396,5 @@
   <axis xyz="0.001375 0.0 -0.999999"/>
 </joint>
-<joint name="Revolute 3" type="continuous">
+<joint name="back_right_steer" type="continuous">
   <origin xyz="-0.371732 -0.24115 0.231126" rpy="0 0 0"/>
   <parent link="base_link"/>
@@ -402,5 +402,5 @@
   <axis xyz="-0.001415 0.0 -0.999999"/>
 </joint>
-<joint name="Revolute 4" type="continuous">
+<joint name="back_left_steer" type="continuous">
   <origin xyz="-0.372163 0.24115 0.231127" rpy="0 0 0"/>
   <parent link="base_link"/>
@@ -408,5 +408,5 @@
   <axis xyz="-0.001415 0.0 -0.999999"/>
 </joint>
-<joint name="Revolute 5" type="continuous">
+<joint name="front_right_drive" type="continuous">
   <origin xyz="0.000261 0.020556 -0.13" rpy="0 0 0"/>
   <parent link="wheel_steer_v2_1"/>
@@ -414,5 +414,5 @@
   <axis xyz="0.0 -1.0 -0.0"/>
 </joint>
-<joint name="Revolute 6" type="continuous">
+<joint name="front_left_drive" type="continuous">
   <origin xyz="0.000179 -0.020557 -0.13" rpy="0 0 0"/>
   <parent link="wheel_steer_v2_2"/>
@@ -420,5 +420,5 @@
   <axis xyz="-0.0 1.0 0.0"/>
 </joint>
-<joint name="Revolute 7" type="continuous">
+<joint name="back_left_drive" type="continuous">
   <origin xyz="-0.000183 -0.020557 -0.13" rpy="0 0 0"/>
   <parent link="wheel_steer_v2_4"/>
@@ -426,5 +426,5 @@
   <axis xyz="-0.0 1.0 0.0"/>
 </joint>
-<joint name="Revolute 8" type="continuous">
+<joint name="back_right_drive" type="continuous">
   <origin xyz="-0.000184 0.020556 -0.13" rpy="0 0 0"/>
   <parent link="wheel_steer_v2_3"/>
@@ -447,5 +447,5 @@
   <child link="base_arm_v2_1"/>
 </joint>
-<joint name="Revolute 12" type="continuous">
+<joint name="base_twist" type="continuous">
   <origin xyz="0.01 0.01 0.041" rpy="0 0 0"/>
   <parent link="base_arm_v2_1"/>
@@ -453,5 +453,5 @@
   <axis xyz="-0.0 0.0 -1.0"/>
 </joint>
-<joint name="Revolute 13" type="continuous">
+<joint name="shoulder" type="continuous">
   <origin xyz="-0.005962 0.041051 0.07474" rpy="0 0 0"/>
   <parent link="link_1_v3_1"/>
@@ -459,5 +459,5 @@
   <axis xyz="1.0 0.0 -0.0"/>
 </joint>
-<joint name="Revolute 14" type="continuous">
+<joint name="elbow" type="continuous">
   <origin xyz="0.0 0.119401 0.1194" rpy="0 0 0"/>
   <parent link="link_2_v1_1"/>
@@ -465,5 +465,5 @@
   <axis xyz="1.0 -0.0 -0.0"/>
 </joint>
-<joint name="Revolute 15" type="continuous">
+<joint name="wrist" type="continuous">
   <origin xyz="0.0003 0.090455 0.090456" rpy="0 0 0"/>
   <parent link="link_3_v2_1"/>
@@ -471,5 +471,5 @@
   <axis xyz="-1.0 0.0 0.0"/>
 </joint>
-<joint name="Revolute 16" type="continuous">
+<joint name="left_grip" type="continuous">
   <origin xyz="0.00851 0.053311 0.039936" rpy="0 0 0"/>
   <parent link="eef_base_v1_1"/>
@@ -477,5 +477,5 @@
   <axis xyz="0.0 -0.707107 0.707107"/>
 </joint>
-<joint name="Revolute 17" type="continuous">
+<joint name="right_grip" type="continuous">
   <origin xyz="0.05051 0.038462 0.025087" rpy="0 0 0"/>
   <parent link="eef_base_v1_1"/>

File: agribot_v4_description/urdf/materials.xacro (robot description, xacro)
@@ -7,6 +7,6 @@
   <color rgba="0.6274509803921569 0.6274509803921569 0.6274509803921569 1.0"/>
 </material>
-<material name="opaque636363">
-  <color rgba="0.25098039215686274 0.25098039215686274 0.25098039215686274 1.0"/>
+<material name="opaque272727">
+  <color rgba="0.10588235294117647 0.10588235294117647 0.10588235294117647 1.0"/>
 </material>
 </robot>

Commit message: Add files via upload

File: agribot_v4_description/urdf/agribot_v4.xacro (robot description, xacro)
@@ -224,4 +224,18 @@
   </collision>
 </link>
+<link name="rgb_frame"/>
+<joint name="kinect_rgb_frame" type="fixed">
+  <parent link="kinectv2_v1_1"/>
+  <child link="rgb_frame"/>
+  <origin xyz="0.075 0.00 0.0375" rpy="0 0 2.61799"/>
+  <axis xyz="0 0 0"/>
+</joint>
+<link name="optical_frame"/>
+<joint name="rgb_optical_frame" type="fixed">
+  <parent link="rgb_frame"/>
+  <child link="optical_frame"/>
+  <origin xyz="0 0 0" rpy="-1.5708 0 -1.5708"/>
+  <axis xyz="0 0 0"/>
+</joint>
 <link name="base_arm_v2_1">
   <inertial>
@@ -371,5 +385,5 @@
   </inertial>
   <visual>
-    <origin xyz="0.25 0.0 -0.555912" rpy="0 0 0"/>
+    <origin xyz="0.25 0.0 -0.585912" rpy="0 0 0"/>
     <geometry>
       <mesh filename="package://agribot_v4_description/meshes/ydlidar_x4_v1_1.stl" scale="0.001 0.001 0.001"/>
@@ -484,5 +498,5 @@
 </joint>
 <joint name="Rigid 18" type="fixed">
-  <origin xyz="-0.25 0.0 0.555912" rpy="0 0 0"/>
+  <origin xyz="-0.25 0.0 0.585912" rpy="0 0 0"/>
   <parent link="base_link"/>
   <child link="ydlidar_x4_v1_1"/>

Commit message: Add files via upload

File: agribot_v4_description/urdf/agribot_v4.xacro (robot description, xacro)
@@ -426,5 +426,5 @@
   <parent link="wheel_steer_v2_1"/>
   <child link="wheel_attachment_v5_1"/>
-  <axis xyz="0.0 -1.0 -0.0"/>
+  <axis xyz="0.0 1.0 -0.0"/>
 </joint>
 <joint name="front_left_drive" type="continuous">
@@ -444,5 +444,5 @@
   <parent link="wheel_steer_v2_3"/>
   <child link="wheel_attachment_v5_4"/>
-  <axis xyz="0.0 -1.0 -0.0"/>
+  <axis xyz="0.0 1.0 -0.0"/>
 </joint>
 <joint name="Rigid 9" type="fixed">
@@ -486,5 +486,5 @@
 </joint>
 <joint name="left_grip" type="continuous">
-  <origin xyz="0.00851 0.053311 0.039936" rpy="0 0 0"/>
+  <origin xyz="-0.01249 0.038462 0.025087" rpy="0 0 0"/>
   <parent link="eef_base_v1_1"/>
   <child link="left_claw_v3_1"/>
